Commit message: Measure the real robot and put the numbers into the model
Everything downstream of the simulated robot -- the policies, the action
scale, the crank zero -- was resting on estimates. This measures what could
be measured and replaces the guesses, adding RobotParams.asbuilt() as the
single place those numbers live.

What the measurements changed:

  legs          20 g -> 9 g    Printed parts are sparse-infill, so mesh
                               volume times material density overestimates
                               them badly. Leg inertia dominates the swing,
                               so this matters more than the 2 percent error
                               in the 303.9 g total.
  servo_kp      5.0 -> 0.673   Identified by matching simulated step
  rotor inertia 1e-8 -> 2.3e-8 responses to ten measured ones (5 to 120
  damping       0.048 -> 0.055 degrees, both directions). Trajectory error
  frictionloss  0 -> 0.00877   fell from 17.0% to 2.5%, and on the other
                               leg's step -- held out of the fit -- from
                               3.74 to 0.32 deg RMS.
  floor         1.0 -> 0.302   Shoved along the floor it runs on, reading
                               the tilt of the specific force while sliding.

Dry friction is new rather than adjusted: with torque off the leg does not
fall at all, so friction exceeds the 1.5e-3 N.m gravity applies to it, and a
viscous-only joint cannot reproduce that. joint_damping stops being derived
as stall torque over no-load speed, which describes the motor's electrical
behaviour rather than mechanical drag.

The tools are kept because these all want re-measuring when the hardware
changes: scripts/mirror mirrors the robot into MuJoCo live, which is how the
conventions were settled; imu_calib finds the IMU's mounting rotation (4.6
degrees off axis-aligned, reproduced across runs, so real); friction_test
measures the floor without needing to tilt it.

Co-Authored-By: Claude Opus 5 <noreply@anthropic.com>

File: hardware/goron.urdf (robot description, URDF)
Before this commit: robot goron, 3 links, 2 joints
Links:
- link base_link: mass 0.27000 -> 0.28590
- link leg_left: mass 0.02000 -> 0.00900
- link leg_right: mass 0.02000 -> 0.00900
